Commit message: Fix Gazebo leg-swing demo with symmetric stand and larger joint swing.
Anchor base via world fixed joint, disable link gravity, unify left/right
initial pose, and drive alternating lifts with calibrated joint-space motion.

Co-authored-by: Cursor <cursoragent@cursor.com>

File: src/biped2_description/urdf/biped2.urdf.xacro (robot description, xacro)
@@ -1,4 +1,6 @@
 <?xml version="1.0"?>
 <robot xmlns:xacro="http://www.ros.org/wiki/xacro" name="biped2">
+  <!-- Anchor base_link in mid-air for leg-swing demo -->
+  <link name="world"/>
 <link
     name="base_link">
@@ -581,22 +583,53 @@
     <limit lower="-0.8" upper="0.8" effort="8" velocity="10" />
   </joint>
+  <joint name="world_to_base_fixed" type="fixed">
+    <parent link="world"/>
+    <child link="base_link"/>
+    <origin xyz="0 0 0.65" rpy="0 0 0"/>
+  </joint>
+  <gazebo reference="world_to_base_fixed">
+    <preserveFixedJoint>true</preserveFixedJoint>
+  </gazebo>
+  <!-- Demo mode: no gravity on links; legs move only via joint trajectory -->
   <gazebo reference="base_link">
     <gravity>false</gravity>
   </gazebo>
-  <!-- Standing pose: feet near ground when base_link is spawned at z=0.45 -->
+  <gazebo reference="RightHipYaw_Link"><gravity>false</gravity></gazebo>
+  <gazebo reference="RightHipRoll_Link"><gravity>false</gravity></gazebo>
+  <gazebo reference="RightHipPitch_Link"><gravity>false</gravity></gazebo>
+  <gazebo reference="RightKneePitch_Link"><gravity>false</gravity></gazebo>
+  <gazebo reference="RightAnklePitch_Link"><gravity>false</gravity></gazebo>
+  <gazebo reference="LeftHipYaw_Link"><gravity>false</gravity></gazebo>
+  <gazebo reference="LeftHipRoll_Link"><gravity>false</gravity></gazebo>
+  <gazebo reference="LeftHipPitch_Link"><gravity>false</gravity></gazebo>
+  <gazebo reference="LeftKneePitch_Link"><gravity>false</gravity></gazebo>
+  <gazebo reference="LeftAnklePitch_Link"><gravity>false</gravity></gazebo>
+  <!-- Symmetric standing pose: both feet at the same height -->
+  <gazebo reference="LeftHipYaw">
+    <initialPosition>0.0</initialPosition>
+  </gazebo>
+  <gazebo reference="LeftHipRoll">
+    <initialPosition>0.0</initialPosition>
+  </gazebo>
   <gazebo reference="LeftHipPitch">
-    <initialPosition>0.4</initialPosition>
+    <initialPosition>0.0155</initialPosition>
   </gazebo>
   <gazebo reference="LeftKneePitch">
-    <initialPosition>-0.8</initialPosition>
+    <initialPosition>-0.0268</initialPosition>
   </gazebo>
   <gazebo reference="LeftAnklePitch">
     <initialPosition>0.4</initialPosition>
   </gazebo>
+  <gazebo reference="RightHipYaw">
+    <initialPosition>0.0</initialPosition>
+  </gazebo>
+  <gazebo reference="RightHipRoll">
+    <initialPosition>0.0</initialPosition>
+  </gazebo>
   <gazebo reference="RightHipPitch">
-    <initialPosition>0.4</initialPosition>
+    <initialPosition>-0.0155</initialPosition>
   </gazebo>
   <gazebo reference="RightKneePitch">
-    <initialPosition>-0.8</initialPosition>
+    <initialPosition>0.0268</initialPosition>
   </gazebo>
   <gazebo reference="RightAnklePitch">

Commit message: Add cycloid alternating leg-swing demo with flat soles and Chinese README.
Drive both legs with half-cycle offset cycloid foot IK, keep soles level,
and document installation plus architecture in the workspace README.

Co-authored-by: Cursor <cursoragent@cursor.com>

File: src/biped2_description/urdf/biped2.urdf.xacro (robot description, xacro)
@@ -1,4 +1,6 @@
 <?xml version="1.0"?>
 <robot xmlns:xacro="http://www.ros.org/wiki/xacro" name="biped2">
+  <!-- Robot height: base_link z in world frame. ~0.37 m puts feet near ground (z=0). -->
+  <xacro:property name="base_height" value="0.37"/>
   <!-- Anchor base_link in mid-air for leg-swing demo -->
   <link name="world"/>
@@ -586,5 +588,5 @@
     <parent link="world"/>
     <child link="base_link"/>
-    <origin xyz="0 0 0.65" rpy="0 0 0"/>
+    <origin xyz="0 0 ${base_height}" rpy="0 0 0"/>
   </joint>
   <gazebo reference="world_to_base_fixed">
@@ -619,5 +621,5 @@
   </gazebo>
   <gazebo reference="LeftAnklePitch">
-    <initialPosition>0.4</initialPosition>
+    <initialPosition>0.0</initialPosition>
   </gazebo>
   <gazebo reference="RightHipYaw">
@@ -634,5 +636,5 @@
   </gazebo>
   <gazebo reference="RightAnklePitch">
-    <initialPosition>0.4</initialPosition>
+    <initialPosition>0.0</initialPosition>
   </gazebo>
   <gazebo>
